File: kicad/wyostat.sch (KiCad schematic (older format))
At the start: 0 parts

Commit message: kicad schematic, WIP
Parts:
- added C? (x3): 100nF,630V, symbol KlokTHREEjr:C_NP
- added D? (x3): LED, symbol KlokTHREEjr:LED
- added J? (x4): Conn_01x02, symbol Connector_Generic:Conn_01x02
- added Q? (x3): BT136-600, TO_SOT_Packages_THT:TO-220_Neutral123_Vertical, symbol wyostat:BT136-600
- added R? (x9): 180, symbol wyostat:R
- added R? (x3): 2k4, symbol wyostat:R
- added U? (x3): MOC3063M, symbol wyostat:MOC3063M
- added U?: Wemos-Lolin, symbol wyostat:Wemos-Lolin
Connections:
- net labels added: GND, IN1, IN2, IN3, LINE, NEUT, OUT1, OUT2, OUT3
- wire segments 0 -> 71
Other:
- note added: "BOM :\n1. ESP32 : Wemos Lolin\n2. Opto : MOC3063SR2M\n3. Triac : BT134-600E,127"

Commit message: schematic WIP
Parts:
- added C? (x2): 100nF, KlokTHREEjr_libs:c_0805, symbol KlokTHREEjr:C_NP
- added C?: C_NP, symbol KlokTHREEjr:C_NP
- added C?: C_POL, symbol KlokTHREEjr:C_POL
- added C? (x3): 10nF,630V, symbol KlokTHREEjr:C_NP
- added D?: DiodeBridge, symbol wyostat:DiodeBridge
- added F?: Polyfuse, symbol wyostat:Polyfuse
- added J?: SPI, KlokTHREEjr_libs:Header_ISP, symbol KlokTHREEjr:Conn_02x03_Odd_Even
- added J?: MISO, KlokTHREEjr_libs:BreakOutPad, symbol KlokTHREEjr:Conn_01x01
- added J?: SCK, KlokTHREEjr_libs:BreakOutPad, symbol KlokTHREEjr:Conn_01x01
- added J?: RST, KlokTHREEjr_libs:BreakOutPad, symbol KlokTHREEjr:Conn_01x01
- added J?: GND, KlokTHREEjr_libs:BreakOutPad, symbol KlokTHREEjr:Conn_01x01
- added J?: MOSI, KlokTHREEjr_libs:BreakOutPad, symbol KlokTHREEjr:Conn_01x01
- added J?: 3V3, KlokTHREEjr_libs:BreakOutPad, symbol KlokTHREEjr:Conn_01x01
- added J?: I2C_ext1, KlokTHREEjr_libs:Header_4x1, symbol KlokTHREEjr:Conn_01x04
- added J?: OUT3, symbol KlokTHREEjr:Conn_01x02
- added JP? (x3): LED1_en, symbol KlokTHREEjr:Jumper_NC_Small
- added R? (x4): 10k, KlokTHREEjr_libs:r_0805, symbol KlokTHREEjr:R
- added R? (x3): 360, symbol wyostat:R
- added R? (x3): 39, symbol wyostat:R
- added S?: SW-DEC, KlokTHREEjr_libs:SW_SMD, symbol KlokTHREEjr:SW-SPST-M
- added S?: SW-MODE, KlokTHREEjr_libs:SW_SMD, symbol KlokTHREEjr:SW-SPST-M
- added S?: SW-ENTER, KlokTHREEjr_libs:SW_SMD, symbol KlokTHREEjr:SW-SPST-M
- added S?: SW-INC, KlokTHREEjr_libs:SW_SMD, symbol KlokTHREEjr:SW-SPST-M
- C? (x3): value 100nF,630V -> 47nF,630V
- J?: value Conn_01x02 -> OUT1; symbol Connector_Generic:Conn_01x02 -> KlokTHREEjr:Conn_01x02; manf# (none) -> Value
- J?: value Conn_01x02 -> PWR_In; symbol Connector_Generic:Conn_01x02 -> KlokTHREEjr:Conn_01x02; manf# (none) -> Value
- J?: value Conn_01x02 -> OUT2; symbol Connector_Generic:Conn_01x02 -> KlokTHREEjr:Conn_01x02; manf# (none) -> Value
- J?: value Conn_01x02 -> OUT3; symbol Connector_Generic:Conn_01x02 -> KlokTHREEjr:Conn_01x02; manf# (none) -> Value
- R? (x3): value 180 -> 360; manf# (none) -> Value
- R? (x3): value 2k4 -> 470; manf# (none) -> Value
- R? (x3): value 180 -> 200; manf# (none) -> Value
- R? (x3): value 180 -> 300; manf# (none) -> Value
Connections:
- net labels added: 3V3, 5V, MISO, MOSI, RST, SCK, SCL, SDA, SW_D, SW_E, SW_I, SW_M
- wire segments 71 -> 213
Other:
- note added: "1.5V/5mA"
- note added: "2V/5mA"
- note added: "BOM :\n1. ESP32 : Wemos Lolin\n2. Opto : MOC3063SR2M\n3. Triac : BT134-600E,127\n4. LED : LTST-C193KGKT-5A\n5. Bridge Rectifier : MDB6S\n6. PTC Fuse : 0ZCF0075AF2C\n7. DC-DC Converter : MAX17502"
- note added: "I2C HEADER"
- note added: "I2C interface for external\nconnections to sensors etc.\n"
- note added: "Native SPI pins are (clk, mosi, miso, cs):\nSPI1: 6, 8, 7, 11\nHSPI: 14,13,12,15\nVSPI: 18,23,19, 5\nIf using native pins max SPI clock can be set to 80 MHZ.\nOnly HSPI & VSPI are supported by esp-idf driver."
- note added: "Push Buttons"
- note added: "SPI HEADER"
- note added: "SPI header with breakout pins.\nConnect with wire to appropriate\npins on ESP32"
- note added: "TRIAC outputs"
- note removed: "BOM :\n1. ESP32 : Wemos Lolin\n2. Opto : MOC3063SR2M\n3. Triac : BT134-600E,127"
- moved on the sheet: Q?, R?, U?

Commit message: kicad schematic, WIP
Parts:
- added C10: 100uF,50V, symbol wyostat:C_POL
- added C11: 2.2uF, symbol wyostat:C_POL
- added C12: 1uF, symbol wyostat:C_NP
- added C13: 3.3nF, symbol wyostat:C_NP
- added J14: ~RST, symbol wyostat:Conn_01x01
- added L1: 22uH, symbol wyostat:L
- added U5: MAX17502FATB+T, TDFN 10, symbol wyostat:MAX17502FATB+T
- C1, C2, C3, C4, C5, C6, C7, C8: renamed from C?; symbol KlokTHREEjr:C_NP -> wyostat:C_NP
- C14: renamed from C?; value C_POL -> 10uF; symbol KlokTHREEjr:C_POL -> wyostat:C_POL
- C9: renamed from C?; value C_NP -> 100nF; symbol KlokTHREEjr:C_NP -> wyostat:C_NP
- D1, D2, D3: renamed from D?; symbol KlokTHREEjr:LED -> wyostat:LED
- J1, J2, J3, J7: renamed from J?; symbol KlokTHREEjr:Conn_01x02 -> wyostat:Conn_01x02
- J10, J11, J12, J5, J6, J8: renamed from J?; symbol KlokTHREEjr:Conn_01x01 -> wyostat:Conn_01x01
- J13: renamed from J?; value OUT3 -> AC_IN; symbol KlokTHREEjr:Conn_01x02 -> wyostat:Conn_01x02
- J4: renamed from J?; symbol KlokTHREEjr:Conn_01x04 -> wyostat:Conn_01x04
- J9: renamed from J?; symbol KlokTHREEjr:Conn_02x03_Odd_Even -> wyostat:Conn_02x03_Odd_Even
- JP1, JP2, JP3: renamed from JP?; value LED1_en -> LED_en; symbol KlokTHREEjr:Jumper_NC_Small -> wyostat:Jumper_NC_Small
- R5, R6, R7, R8: renamed from R?; symbol KlokTHREEjr:R -> wyostat:R
- S1, S2, S3, S4: renamed from S?; symbol KlokTHREEjr:SW-SPST-M -> wyostat:SW-SPST-M
- gave numbers to parts that had none: 27
Connections:
- net labels added: 5V_IN, GNDREF
- wire segments 213 -> 255
- no-connect marks 0 -> 13
Other:
- note added: "AC-DC POWER SUPPLY"
- note added: "Connect GNDREF to GND\nat VCC capacitor"
- note added: "DECIDE how to couple 5V_IN to 5V"
- moved on the sheet: D4, F1, Q1, Q2, Q3, R1, R10, R11, R12, R13, R14, R15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

Commit message: kicad schematic, WIP
Parts:
- C1: value 10nF,630V -> 10nF,250V; footprint (none) -> Capacitors_Tantalum_SMD:CP_Tantalum_Case-E_EIA-7260-38_Hand
- C11, C12, C13, C14, C9: footprint (none) -> Capacitors_SMD:C_0805
- C2, C5, C8: value 47nF,630V -> 47nF,250V
- C3, C6: footprint KlokTHREEjr_libs:c_0805 -> Capacitors_SMD:C_0805
- C4, C7: value 10nF,630V -> 10nF,250V
- D1, D2, D3: footprint (none) -> LEDs:LED_0603
- F1: footprint (none) -> Fuse_Holders_and_Fuses:Fuse_SMD2920
- J1, J13, J2, J3, J7: footprint (none) -> Connectors_Terminal_Blocks:TerminalBlock_Pheonix_MPT-2.54mm_2pol
- J10, J11, J12, J5, J6, J8: footprint KlokTHREEjr_libs:BreakOutPad -> Pin_Headers:Pin_Header_Straight_1x01
- J14: footprint (none) -> Pin_Headers:Pin_Header_Straight_1x01
- J4: footprint KlokTHREEjr_libs:Header_4x1 -> Pin_Headers:Pin_Header_Straight_1x04
- J9: footprint KlokTHREEjr_libs:Header_ISP -> Pin_Headers:Pin_Header_Straight_2x03
- JP1, JP2, JP3: footprint (none) -> LEDs:LED_0402
- R1, R10, R11, R12, R13, R14, R15, R16, R17, R18, R19, R2, R20, R21, R22, R3, R4, R9: footprint (none) -> Resistors_SMD:R_0805
- R5, R6, R7, R8: footprint KlokTHREEjr_libs:r_0805 -> Resistors_SMD:R_0805
- U1, U3, U4: footprint (none) -> Opto-Devices:Optocoupler_6pin_wide_Stile-I
- U5: footprint TDFN 10 -> (none)
Other:
- note added: "BOM :\n1. ESP32 : Wemos Lolin\n2. Opto : MOC3063SR2M\n3. Triac : BT134-600E,127\n4. LED : LTST-C193KGKT-5A\n5. Bridge Rectifier : MDB6S\n6. PTC Fuse : 0ZCF0075AF2C\n7. DC-DC Converter : MAX17502\n8. 10nF,250V : LDEQE2100KA5N00"
- note removed: "BOM :\n1. ESP32 : Wemos Lolin\n2. Opto : MOC3063SR2M\n3. Triac : BT134-600E,127\n4. LED : LTST-C193KGKT-5A\n5. Bridge Rectifier : MDB6S\n6. PTC Fuse : 0ZCF0075AF2C\n7. DC-DC Converter : MAX17502"

Commit message: schematic WIP
Parts:
- C11: value 2.2uF -> 2.2uF,50V
- R10, R15, R22: DNP DNP -> -; manf# (none) -> Value
Changed lines of the file:
@@
 U 1 1 5AA6EEDE
 P 8325 1250
-F 0 "U1" H 8325 1625 50  0000 C CNN
-F 1 "MOC3063M" H 8325 1525 50  0000 C CNN
+F 0 "U1" H 8325 1525 50  0000 C CNN
+F 1 "MOC3063M" H 8350 1450 50  0000 C CNN
 F 2 "Opto-Devices:Optocoupler_6pin_wide_Stile-I" H 8125 1050 50  0001 L CIN
 F 3 "" H 8290 1250 50  0001 L CNN
@@
 U 1 1 5AA72CD7
 P 7675 1300
-F 0 "D1" V 7625 1425 40  0000 L CNN
-F 1 "LED" V 7675 1425 40  0000 L CNN
+F 0 "D1" V 7625 1375 40  0000 L CNN
+F 1 "LED" V 7675 1375 40  0000 L CNN
 F 2 "LEDs:LED_0603" H 7675 1300 60  0001 C CNN
 F 3 "" H 7675 1300 60  0000 C CNN
@@
 U 1 1 5AA791A2
 P 8325 2750
-F 0 "U3" H 8325 3125 50  0000 C CNN
-F 1 "MOC3063M" H 8325 3025 50  0000 C CNN
+F 0 "U3" H 8325 3025 50  0000 C CNN
+F 1 "MOC3063M" H 8325 2950 50  0000 C CNN
 F 2 "Opto-Devices:Optocoupler_6pin_wide_Stile-I" H 8125 2550 50  0001 L CIN
 F 3 "" H 8290 2750 50  0001 L CNN
@@
 U 1 1 5AA791E3
 P 7675 2800
-F 0 "D2" V 7625 2925 40  0000 L CNN
-F 1 "LED" V 7675 2925 40  0000 L CNN
+F 0 "D2" V 7625 2875 40  0000 L CNN
+F 1 "LED" V 7675 2875 40  0000 L CNN
 F 2 "LEDs:LED_0603" H 7675 2800 60  0001 C CNN
 F 3 "" H 7675 2800 60  0000 C CNN
@@
 U 1 1 5AA7ACC5
 P 8325 4250
-F 0 "U4" H 8325 4625 50  0000 C CNN
-F 1 "MOC3063M" H 8325 4525 50  0000 C CNN
+F 0 "U4" H 8325 4525 50  0000 C CNN
+F 1 "MOC3063M" H 8325 4450 50  0000 C CNN
 F 2 "Opto-Devices:Optocoupler_6pin_wide_Stile-I" H 8125 4050 50  0001 L CIN
 F 3 "" H 8290 4250 50  0001 L CNN
@@
 U 1 1 5AA7AD06
 P 7675 4300
-F 0 "D3" V 7625 4425 40  0000 L CNN
-F 1 "LED" V 7675 4425 40  0000 L CNN
+F 0 "D3" V 7625 4375 40  0000 L CNN
+F 1 "LED" V 7675 4375 40  0000 L CNN
 F 2 "LEDs:LED_0603" H 7675 4300 60  0001 C CNN
 F 3 "" H 7675 4300 60  0000 C CNN
@@
 U 1 1 5AA958CA
 P 5675 4125
-F 0 "J9" H 5725 4400 50  0000 C CNN
-F 1 "SPI" H 5725 4325 50  0000 C CNN
+F 0 "J9" H 5725 4325 50  0000 C CNN
+F 1 "SPI" H 5725 3925 50  0000 C CNN
 F 2 "Pin_Headers:Pin_Header_Straight_2x03" H 5675 4125 50  0001 C CNN
 F 3 "~" H 5675 4125 50  0001 C CNN
@@
 U 1 1 5AA95913
 P 5575 2575
-F 0 "J4" H 5525 2775 50  0000 L CNN
-F 1 "I2C_ext1" V 5675 2325 50  0000 L CNN
+F 0 "J4" H 5575 2775 50  0000 C CNN
+F 1 "I2C_ext1" H 5575 2275 50  0000 C CNN
 F 2 "Pin_Headers:Pin_Header_Straight_1x04" H 5575 2575 50  0001 C CNN
 F 3 "~" H 5575 2575 50  0001 C CNN
@@
 Wire Wire Line
 	1275 1075 1375 1075
-Text Notes 7650 1525 2    40   ~ 0
+Text Notes 7650 1500 2    40   ~ 0
 2V/5mA
-Text Notes 7900 1525 0    40   ~ 0
+Text Notes 7875 1500 0    40   ~ 0
 1.5V/5mA
 $Comp
@@
 U 1 1 5AD09F0B
 P 825 5975
-F 0 "J13" H 925 5975 50  0000 L CNN
-F 1 "AC_IN" H 750 5775 50  0000 L CNN
+F 0 "J13" H 825 6100 50  0000 C CNN
+F 1 "AC_IN" H 825 5775 50  0000 C CNN
 F 2 "Connectors_Terminal_Blocks:TerminalBlock_Pheonix_MPT-2.54mm_2pol" H 825 5975 50  0001 C CNN
 F 3 "~" H 825 5975 50  0001 C CNN
@@
 F 2 "Resistors_SMD:R_0805" V 9830 1750 50  0001 C CNN
 F 3 "" H 9900 1750 50  0001 C CNN
-F 4 "DNP" V 9975 1750 30  0000 C CNN "DNP"
+F 4 "Value" H 9900 1750 50  0001 C CNN "manf#"
+F 5 "-" V 9900 1750 50  0001 C CNN "DNP"
 	1    9900 1750
 	-1   0    0    1
@@
 F 2 "Resistors_SMD:R_0805" V 9830 3250 50  0001 C CNN
 F 3 "" H 9900 3250 50  0001 C CNN
-F 4 "DNP" V 9975 3250 30  0000 C CNN "DNP"
+F 4 "Value" H 9900 3250 50  0001 C CNN "manf#"
+F 5 "-" V 9975 3250 30  0001 C CNN "DNP"
 	1    9900 3250
 	-1   0    0    1
@@
 F 2 "Resistors_SMD:R_0805" V 9830 4750 50  0001 C CNN
 F 3 "" H 9900 4750 50  0001 C CNN
-F 4 "DNP" V 9975 4750 30  0000 C CNN "DNP"
+F 4 "Value" H 9900 4750 50  0001 C CNN "manf#"
+F 5 "-" V 9975 4750 30  0001 C CNN "DNP"
 	1    9900 4750
 	-1   0    0    1
@@
 P 2725 7025
 F 0 "C11" H 2750 6925 40  0000 L CNN
-F 1 "2.2uF" V 2775 7150 40  0000 L CNN
+F 1 "2.2uF,50V" V 2775 7150 40  0000 L CNN
 F 2 "Capacitors_SMD:C_0805" H 2725 7025 60  0001 C CNN
 F 3 "" H 2725 7025 60  0000 C CNN
@@
 U 1 1 5AB874BA
 P 5325 6775
-F 0 "J14" H 5450 6850 50  0000 L CNN
-F 1 "~RST" H 5450 6750 50  0000 L CNN
+F 0 "J14" H 5325 6875 50  0000 C CNN
+F 1 "~RST" H 5325 6650 50  0000 C CNN
 F 2 "Pin_Headers:Pin_Header_Straight_1x01" H 5325 6775 50  0001 C CNN
 F 3 "" H 5325 6775 50  0001 C CNN

Commit message: kicad schematic, WIP
Parts:
- C1: footprint Capacitors_Tantalum_SMD:CP_Tantalum_Case-E_EIA-7260-38_Hand -> wyostat_fp:C_2220
- C10, C2, C4, C5, C7, C8: footprint (none) -> wyostat_fp:C_2220
- C11, C12, C13, C14, C3, C6, C9: footprint Capacitors_SMD:C_0805 -> wyostat_fp:C_0805
- D1, D2, D3: footprint LEDs:LED_0603 -> wyostat_fp:LED_0603
- D4: footprint (none) -> wyostat_fp:Diode_bridge
- F1: footprint Fuse_Holders_and_Fuses:Fuse_SMD2920 -> wyostat_fp:Fuse_SMD2920
- J1, J13, J2, J3, J7: footprint Connectors_Terminal_Blocks:TerminalBlock_Pheonix_MPT-2.54mm_2pol -> wyostat_fp:TerminalBlock_Pheonix_MPT-2.54mm_2pol
- J10, J11, J12, J14, J5, J6, J8: footprint Pin_Headers:Pin_Header_Straight_1x01 -> wyostat_fp:Pin_Header_Straight_1x01
- J4: footprint Pin_Headers:Pin_Header_Straight_1x04 -> wyostat_fp:Pin_Header_Straight_1x04
- J9: footprint Pin_Headers:Pin_Header_Straight_2x03 -> wyostat_fp:Pin_Header_Straight_2x03
- JP1, JP2, JP3: footprint LEDs:LED_0402 -> wyostat_fp:LED_0402
- L1: footprint (none) -> wyostat_fp:Inductor_ELL8TP
- Q1, Q2, Q3: footprint TO_SOT_Packages_THT:TO-220_Neutral123_Vertical -> wyostat_fp:SOT126_SOT32_Housing_Horizontal
- R1, R10, R11, R12, R13, R14, R15, R16, R17, R18, R19, R2, R20, R21, R22, R3, R4, R5, R6, R7, R8, R9: footprint Resistors_SMD:R_0805 -> wyostat_fp:R_0805
- S1, S2, S3, S4: footprint KlokTHREEjr_libs:SW_SMD -> wyostat_fp:SW_SPST_CK_KSCx
- U1, U3, U4: footprint Opto-Devices:Optocoupler_6pin_wide_Stile-I -> wyostat_fp:Optocoupler_6pin
- U2: footprint (none) -> wyostat_fp:Wemos_Lolin
- U5: footprint (none) -> wyostat_fp:TDFN-10
Connections:
- net IN1: now also U2.8 (12); no longer U2.6 (2)
- net IN2: now also U2.9 (13); no longer U2.7 (14)
- net IN3: now also U2.10 (15); no longer U2.8 (12)
- net SW_D: now also U2.6 (2); no longer U2.4
- net SW_I: now also U2.5 (0); no longer U2.3 (5)
- net SW_M: now also U2.7 (14); no longer U2.5 (0)
Other:
- note added: "BOM :\n1. ESP32 : Wemos Lolin\n2. Opto : MOC3063SR2M\n3. Triac : BT134-600E,127\n4. LED : LTST-C193KGKT-5A\n5. Bridge Rectifier : MDB6S\n6. PTC Fuse : 0ZCF0075AF2C\n7. DC-DC Converter : MAX17502\n8. 10nF,250V : LDEQE2100KA5N00\n9. Inductor L1 : ELL-8TP220MB"
- note removed: "BOM :\n1. ESP32 : Wemos Lolin\n2. Opto : MOC3063SR2M\n3. Triac : BT134-600E,127\n4. LED : LTST-C193KGKT-5A\n5. Bridge Rectifier : MDB6S\n6. PTC Fuse : 0ZCF0075AF2C\n7. DC-DC Converter : MAX17502\n8. 10nF,250V : LDEQE2100KA5N00"
- moved on the sheet: U2

Commit message: kicad schematic, WIP
Parts:
- C1, C4, C7: value 10nF,250V -> 10nF,100V
- C2, C5, C8: value 47nF,250V -> 47nF,100V
Other:
- note added: "40 V AC MAX"
- note added: "40 V AC MAX."
Changed lines of the file:
@@
 P 9025 1750
 F 0 "C2" H 9050 1850 40  0000 L CNN
-F 1 "47nF,250V" H 9050 1650 40  0000 L CNN
+F 1 "47nF,100V" H 9050 1650 40  0000 L CNN
 F 2 "wyostat_fp:C_2220" H 9025 1750 60  0001 C CNN
 F 3 "" H 9025 1750 60  0000 C CNN
@@
 P 9025 3300
 F 0 "C5" H 9050 3400 40  0000 L CNN
-F 1 "47nF,250V" H 9050 3200 40  0000 L CNN
+F 1 "47nF,100V" H 9050 3200 40  0000 L CNN
 F 2 "wyostat_fp:C_2220" H 9025 3300 60  0001 C CNN
 F 3 "" H 9025 3300 60  0000 C CNN
@@
 P 9025 4750
 F 0 "C8" H 9050 4850 40  0000 L CNN
-F 1 "47nF,250V" H 9050 4650 40  0000 L CNN
+F 1 "47nF,100V" H 9050 4650 40  0000 L CNN
 F 2 "wyostat_fp:C_2220" H 9025 4750 60  0001 C CNN
 F 3 "" H 9025 4750 60  0000 C CNN
@@
 P 9900 1400
 F 0 "C1" H 9925 1500 40  0000 L CNN
-F 1 "10nF,250V" H 9925 1300 40  0000 L CNN
+F 1 "10nF,100V" H 9925 1300 40  0000 L CNN
 F 2 "wyostat_fp:C_2220" H 9900 1400 60  0001 C CNN
 F 3 "" H 9900 1400 60  0000 C CNN
@@
 P 9900 2900
 F 0 "C4" H 9925 3000 40  0000 L CNN
-F 1 "10nF,250V" H 9925 2800 40  0000 L CNN
+F 1 "10nF,100V" H 9925 2800 40  0000 L CNN
 F 2 "wyostat_fp:C_2220" H 9900 2900 60  0001 C CNN
 F 3 "" H 9900 2900 60  0000 C CNN
@@
 P 9900 4400
 F 0 "C7" H 9925 4500 40  0000 L CNN
-F 1 "10nF,250V" H 9925 4300 40  0000 L CNN
+F 1 "10nF,100V" H 9925 4300 40  0000 L CNN
 F 2 "wyostat_fp:C_2220" H 9900 4400 60  0001 C CNN
 F 3 "" H 9900 4400 60  0000 C CNN
@@
 EndData
 $EndBitmap
+Text Notes 700  6325 0    50   ~ 0
+40 V AC MAX.
+Text Notes 9675 775  0    50   ~ 0
+40 V AC MAX
 $EndSCHEMATC

Commit message: schematic WIP
Parts:
- added F2: Polyfuse, wyostat_fp:Fuse_SMD2920, symbol wyostat:Polyfuse
- added J15: AC_IN, wyostat_fp:TerminalBlock_Pheonix_MPT-2.54mm_2pol, symbol wyostat:Conn_01x02
- added J16: 5V_SEL, symbol wyostat:Conn_01x04
- added U6: Converter_AC_DC, symbol wyostat:Converter_AC_DC
- C1: value 10nF,100V -> 10nF,120V
- C10: footprint wyostat_fp:C_2220 -> Capacitors_SMD:CP_Elec_10x10
- C2: value 47nF,100V -> 47nF,63V
- C3: renamed from C4; value 10nF,100V -> 10nF,120V
- C4: renamed from C5; value 47nF,100V -> 47nF,63V
- C5: renamed from C7; value 10nF,100V -> 10nF,120V
- C6: renamed from C8; value 47nF,100V -> 47nF,63V
- Q1, Q2, Q3: footprint wyostat_fp:SOT126_SOT32_Housing_Horizontal -> SMD_Packages:DPAK-2
- renumbered C3 to C7, C6 to C8, J7 to J4, J4 to J5, J5 to J6, J6 to J7, R14 to R10, R15 to R11, R16 to R12, R17 to R13, R18 to R14, R19 to R15, R20 to R16, R21 to R17, R22 to R18, R5 to R19, R6 to R20, R7 to R21, R8 to R22, R9 to R5, R10 to R6, R11 to R7, R12 to R8, R13 to R9, U3 to U2, U4 to U3, U2 to U4
Connections:
- net 5V: now also J16.2 (Pin_2), J16.3 (Pin_3)
- net GND: now also U6.4 (V-)
- net IN1: now also U4.2 (16); no longer U4.8 (12)
- net IN2: now also U4.25; no longer U4.9 (13)
- net IN3: now also U4.24 (26); no longer U4.10 (15)
- net SCL: now also U4.4
- net SDA: now also U4.3 (5)
- net SW_D: now also U4.8 (12); no longer U4.6 (2)
- net SW_E: now also U4.10 (15); no longer U4.2 (16)
- net SW_I: now also U4.9 (13); no longer U4.5 (0)
- net 5V_IN renamed 5V_IN1
- net 5V_IN1: now also J16.4 (Pin_4)
- new net: F2.1, U6.1 (AC/L)
- new net: J15.2 (Pin_2), U6.2 (AC/N)
- new net: F2.2, J15.1 (Pin_1)
- new net 5V_IN2: J16.1 (Pin_1), U6.3 (V+)
- no-connect marks 13 -> 11
Other:
- note added: "250 V AC MAX."
- note added: "40 V AC MAX.\nISOLATED"
- note added: "BOM :\n1. ESP32 : Wemos Lolin\n2. Opto : MOC3063SR2M\n3. Triac : BT134-600E,127 (TH)\n : BTA204S-600E,118 (SMD)\n4. LED : LTST-C193KGKT-5A\n5. Bridge Rectifier : MDB6S\n6. PTC Fuse : 0ZCF0075AF2C\n7. DC-DC Converter : MAX17502\n8. 10nF/120V AC : LDEIB2100KA0N00\n9. 47nF/63V AC : LDEEB2470KA0N00\n10. Inductor L1 : ELL-8TP220MB\n11. 100uF/50V Elco : HHXC500ARA101MJA0G\n : EMZA630ADA101MJA0G"
- note added: "Connect\nGNDREF to GND\nat VCC capacitor"
- note removed: "40 V AC MAX."
- note removed: "BOM :\n1. ESP32 : Wemos Lolin\n2. Opto : MOC3063SR2M\n3. Triac : BT134-600E,127\n4. LED : LTST-C193KGKT-5A\n5. Bridge Rectifier : MDB6S\n6. PTC Fuse : 0ZCF0075AF2C\n7. DC-DC Converter : MAX17502\n8. 10nF,250V : LDEQE2100KA5N00\n9. Inductor L1 : ELL-8TP220MB"
- note removed: "Connect GNDREF to GND\nat VCC capacitor"
- moved on the sheet: C10, C11, C12, C13, C14, C3, C4, C5, C6, C9, D2, D3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
