File: kicad/wyostat.sch (KiCad schematic (older format))
At the start: 75 parts, among them J1 PWR_In, J10 MOSI, J11 RST, J12 GND, J13 AC_IN, J14 ~RST, J15 AC_IN, J16 5V_SEL, J2 OUT1, J3 OUT2, J4 OUT3, J5 I2C_ext1, J6 MISO, J7 3V3, J8 SCK, J9 SPI, Q1 BT136-600, Q2 BT136-600, Q3 BT136-600, U1 MOC3063M, U2 MOC3063M, U3 MOC3063M, U4 Wemos-Lolin, U5 MAX17502FATB+T, U6 Converter_AC_DC

Commit message: layou, WIP
Parts:
- J16: footprint (none) -> wyostat_fp:Pin_Header_Straight_1x04
- U6: footprint (none) -> wyostat_fp:Converter_AC_DC
Changed lines of the file:
@@
 F 0 "U6" H 1775 5800 40  0000 C CNN
 F 1 "Converter_AC_DC" H 1775 5400 40  0000 C CNN
-F 2 "" H 1725 5600 40  0001 C CNN
+F 2 "wyostat_fp:Converter_AC_DC" H 1725 5600 40  0001 C CNN
 F 3 "" H 1725 5600 40  0001 C CNN
 	1    1775 5600
@@
 F 0 "J16" H 4775 5250 50  0000 C CNN
 F 1 "5V_SEL" V 4875 5500 50  0000 C CNN
-F 2 "" H 4775 5550 50  0001 C CNN
+F 2 "wyostat_fp:Pin_Header_Straight_1x04" H 4775 5550 50  0001 C CNN
 F 3 "" H 4775 5550 50  0001 C CNN
 	1    4775 5550

Commit message: kicad PCB, WIP
Parts:
- removed J14: ~RST, wyostat_fp:Pin_Header_Straight_1x01, symbol wyostat:Conn_01x01
Connections:
- wire segments 287 -> 286
- no-connect marks 11 -> 12
Changed lines of the file:
@@
 L wyostat:Conn_01x02 J13
 U 1 1 5AD09F0B
-P 775 6575
-F 0 "J13" H 775 6700 50  0000 C CNN
-F 1 "AC_IN" H 775 6375 50  0000 C CNN
-F 2 "wyostat_fp:TerminalBlock_Pheonix_MPT-2.54mm_2pol" H 775 6575 50  0001 C CNN
-F 3 "~" H 775 6575 50  0001 C CNN
-F 4 "Value" H 775 6575 50  0001 C CNN "manf#"
-	1    775  6575
-	-1   0    0    -1
+P 775 6675
+F 0 "J13" H 775 6800 50  0000 C CNN
+F 1 "AC_IN" H 775 6475 50  0000 C CNN
+F 2 "wyostat_fp:TerminalBlock_Pheonix_MPT-2.54mm_2pol" H 775 6675 50  0001 C CNN
+F 3 "~" H 775 6675 50  0001 C CNN
+F 4 "Value" H 775 6675 50  0001 C CNN "manf#"
+	1    775  6675
+	-1   0    0    1
 $EndComp
 $Comp
@@
 	3725 7275 3725 7325
 Wire Wire Line
-	4325 7075 4525 7075
-$Comp
-L wyostat:Conn_01x01 J14
-U 1 1 5AB874BA
-P 4725 7075
-F 0 "J14" H 4725 7175 50  0000 C CNN
-F 1 "~RST" H 4725 6950 50  0000 C CNN
-F 2 "wyostat_fp:Pin_Header_Straight_1x01" H 4725 7075 50  0001 C CNN
-F 3 "" H 4725 7075 50  0001 C CNN
-	1    4725 7075
-	1    0    0    -1
-$EndComp
-Wire Wire Line
 	4325 6675 4400 6675
 Wire Wire Line
@@
 Text Notes 700  5875 0    50   ~ 0
 250 V AC MAX.
+NoConn ~ 4325 7075
 $EndSCHEMATC

Commit message: layou, WIP
Parts:
- added JP4: GND, wyostat_fp:LED_0402, symbol wyostat:Jumper_NC_Small
- added SC1, SC2, SC3, SC4: SCREW, wyostat_fp:MountingHole_3.2mm_M3_Pad_Via, symbol wyostat:SCREW
Connections:
- net labels added: 40VDC, LX, R, SS, VCC
- wire segments 286 -> 288
Other:
- note added: "INPUT POWER\n\nInput Power sources are :\na. Micro USB 5V to Wemos Lolin\nb. 28 V AC converted to 5 V via switching regulator\nc. 115 V AC converted to 5 V via wall wart or switching regulator\n\nWhen using option "b" or "c", the micro USB cable\nMUST be removed to prevent power conflicts."
- moved on the sheet: J2, J3, J4
Changed lines of the file:
@@
 	0    1    1    0
 $EndComp
-Text Label 10325 1050 0    40   ~ 0
-LINE
-Text Label 10325 1150 0    40   ~ 0
+Text Label 10325 2025 0    40   ~ 0
 OUT1
-Text Label 9550 2025 2    40   ~ 0
-NEUT
 $Comp
 L wyostat:R R2
@@
 Wire Wire Line
 	9550 1150 9900 1150
-Wire Wire Line
-	10475 1050 10225 1050
 $Comp
 L wyostat:Conn_01x02 J2
 U 1 1 5AA726AC
-P 10675 1050
-F 0 "J2" H 10775 1050 50  0000 L CNN
-F 1 "OUT1" H 10775 950 50  0000 L CNN
-F 2 "wyostat_fp:TerminalBlock_Pheonix_MPT-2.54mm_2pol" H 10675 1050 50  0001 C CNN
-F 3 "~" H 10675 1050 50  0001 C CNN
-F 4 "Value" H 10675 1050 50  0001 C CNN "manf#"
-	1    10675 1050
-	1    0    0    -1
+P 10675 2025
+F 0 "J2" H 10775 2025 50  0000 L CNN
+F 1 "OUT1" H 10775 1925 50  0000 L CNN
+F 2 "wyostat_fp:TerminalBlock_Pheonix_MPT-2.54mm_2pol" H 10675 2025 50  0001 C CNN
+F 3 "~" H 10675 2025 50  0001 C CNN
+F 4 "Value" H 10675 2025 50  0001 C CNN "manf#"
+	1    10675 2025
+	1    0    0    1
 $EndComp
 $Comp
@@
 	0    1    1    0
 $EndComp
-Text Label 10325 2400 0    40   ~ 0
-LINE
-Text Label 10325 2500 0    40   ~ 0
+Text Label 10325 3375 0    40   ~ 0
 OUT2
-Text Label 9550 3375 2    40   ~ 0
-NEUT
 $Comp
 L wyostat:R R8
@@
 Wire Wire Line
 	9550 2500 9900 2500
-Wire Wire Line
-	10475 2400 10225 2400
 $Comp
 L wyostat:Conn_01x02 J3
 U 1 1 5AA791CF
-P 10675 2400
-F 0 "J3" H 10775 2400 50  0000 L CNN
-F 1 "OUT2" H 10775 2300 50  0000 L CNN
-F 2 "wyostat_fp:TerminalBlock_Pheonix_MPT-2.54mm_2pol" H 10675 2400 50  0001 C CNN
-F 3 "~" H 10675 2400 50  0001 C CNN
-F 4 "Value" H 10675 2400 50  0001 C CNN "manf#"
-	1    10675 2400
-	1    0    0    -1
+P 10675 3375
+F 0 "J3" H 10775 3375 50  0000 L CNN
+F 1 "OUT2" H 10775 3275 50  0000 L CNN
+F 2 "wyostat_fp:TerminalBlock_Pheonix_MPT-2.54mm_2pol" H 10675 3375 50  0001 C CNN
+F 3 "~" H 10675 3375 50  0001 C CNN
+F 4 "Value" H 10675 3375 50  0001 C CNN "manf#"
+	1    10675 3375
+	1    0    0    1
 $EndComp
 $Comp
@@
 	0    1    1    0
 $EndComp
-Text Label 10325 3750 0    40   ~ 0
-LINE
-Text Label 10325 3850 0    40   ~ 0
+Text Label 10325 4725 0    40   ~ 0
 OUT3
-Text Label 9550 4725 2    40   ~ 0
-NEUT
 $Comp
 L wyostat:R R14
@@
 L wyostat:Conn_01x02 J4
 U 1 1 5AA7ACF2
-P 10675 3750
-F 0 "J4" H 10775 3750 50  0000 L CNN
-F 1 "OUT3" H 10775 3650 50  0000 L CNN
-F 2 "wyostat_fp:TerminalBlock_Pheonix_MPT-2.54mm_2pol" H 10675 3750 50  0001 C CNN
-F 3 "~" H 10675 3750 50  0001 C CNN
-F 4 "Value" H 10675 3750 50  0001 C CNN "manf#"
-	1    10675 3750
-	1    0    0    -1
+P 10675 4725
+F 0 "J4" H 10775 4725 50  0000 L CNN
+F 1 "OUT3" H 10775 4625 50  0000 L CNN
+F 2 "wyostat_fp:TerminalBlock_Pheonix_MPT-2.54mm_2pol" H 10675 4725 50  0001 C CNN
+F 3 "~" H 10675 4725 50  0001 C CNN
+F 4 "Value" H 10675 4725 50  0001 C CNN "manf#"
+	1    10675 4725
+	1    0    0    1
 $EndComp
 $Comp
@@
 Wire Wire Line
 	7675 3850 8025 3850
-Wire Wire Line
-	10125 800  10125 2025
-Wire Wire Line
-	10125 4725 9900 4725
-Wire Wire Line
-	10125 800  10475 800
 Connection ~ 9550 4725
 Wire Wire Line
 	9550 3375 9900 3375
 Connection ~ 9550 3375
-Connection ~ 10125 3375
-Wire Wire Line
-	10125 3375 10125 4725
 Wire Wire Line
 	9550 2025 9900 2025
 Connection ~ 9550 2025
-Connection ~ 10125 2025
-Wire Wire Line
-	10125 2025 10125 3375
-Wire Wire Line
-	10225 700  10225 1050
-Wire Wire Line
-	10225 700  10475 700
-Wire Wire Line
-	10225 3750 10475 3750
-Connection ~ 10225 2400
-Wire Wire Line
-	10225 2400 10225 3750
-Connection ~ 10225 1050
-Wire Wire Line
-	10225 1050 10225 2400
 Wire Notes Line
 	6925 575  11125 575
@@
 L wyostat:Conn_01x02 J13
 U 1 1 5AD09F0B
-P 775 6675
-F 0 "J13" H 775 6800 50  0000 C CNN
-F 1 "AC_IN" H 775 6475 50  0000 C CNN
-F 2 "wyostat_fp:TerminalBlock_Pheonix_MPT-2.54mm_2pol" H 775 6675 50  0001 C CNN
-F 3 "~" H 775 6675 50  0001 C CNN
-F 4 "Value" H 775 6675 50  0001 C CNN "manf#"
-	1    775  6675
-	-1   0    0    1
+P 775 6575
+F 0 "J13" H 775 6700 50  0000 C CNN
+F 1 "AC_IN" H 775 6375 50  0000 C CNN
+F 2 "wyostat_fp:TerminalBlock_Pheonix_MPT-2.54mm_2pol" H 775 6575 50  0001 C CNN
+F 3 "~" H 775 6575 50  0001 C CNN
+F 4 "Value" H 775 6575 50  0001 C CNN "manf#"
+	1    775  6575
+	-1   0    0    -1
 $EndComp
 $Comp
@@
 Wire Wire Line
 	9900 1250 9900 1150
-Connection ~ 9900 1150
-Wire Wire Line
-	9900 1150 10475 1150
 Wire Wire Line
 	9900 1550 9900 1600
@@
 	9900 1900 9900 2025
 Connection ~ 9900 2025
-Wire Wire Line
-	9900 2025 10125 2025
 $Comp
 L wyostat:C_NP C3
@@
 Wire Wire Line
 	9900 3250 9900 3375
-Connection ~ 9900 2500
-Wire Wire Line
-	9900 2500 10475 2500
 Connection ~ 9900 3375
-Wire Wire Line
-	9900 3375 10125 3375
 $Comp
 L wyostat:C_NP C5
@@
 Wire Wire Line
 	9900 4600 9900 4725
-Connection ~ 9900 3850
-Wire Wire Line
-	9900 3850 10475 3850
 Connection ~ 9900 4725
 Wire Wire Line
@@
 	4325 6475 4475 6475
 Wire Wire Line
-	4475 6475 4475 7475
-Wire Wire Line
-	4475 7475 2650 7475
+	4475 6475 4475 7625
 Wire Wire Line
-	2525 7225 2525 7475
+	2525 7225 2525 7625
 Text Label 2125 7325 0    40   ~ 0
 GND
-Text Label 2825 7325 0    40   ~ 0
+Text Label 3100 7325 0    40   ~ 0
 GND
 $Comp
@@
 L wyostat:GNDREF #PWR03
 U 1 1 5ABDBAC8
-P 2650 7550
-F 0 "#PWR03" H 2650 7300 50  0001 C CNN
-F 1 "GNDREF" H 2475 7550 50  0000 C CNN
-F 2 "" H 2650 7550 50  0001 C CNN
-F 3 "" H 2650 7550 50  0001 C CNN
-	1    2650 7550
+P 5100 7500
+F 0 "#PWR03" H 5100 7250 50  0001 C CNN
+F 1 "GNDREF" H 5275 7500 50  0000 C CNN
+F 2 "" H 5100 7500 50  0001 C CNN
+F 3 "" H 5100 7500 50  0001 C CNN
+	1    5100 7500
 	1    0    0    -1
 $EndComp
 Wire Wire Line
-	4975 7225 4975 7475
+	4975 7225 4975 7400
 Wire Wire Line
-	4975 7475 4475 7475
-Connection ~ 4475 7475
+	4975 7625 4475 7625
+Connection ~ 4475 7625
 $Comp
 L wyostat:L L1
@@
 $EndComp
 Wire Wire Line
-	2750 7325 2650 7400
-Wire Wire Line
-	2650 7400 2650 7475
-Connection ~ 2650 7475
-Wire Wire Line
-	2650 7475 2525 7475
-Wire Wire Line
 	2075 7600 2075 7325
-Wire Wire Line
-	2650 7550 2650 7475
 Text Notes 1550 7575 0    40   ~ 0
 Connect\nGNDREF to GND\nat VCC capacitor
@@
 	2975 7325 2750 7325
 Connection ~ 2975 7325
-Connection ~ 2750 7325
 Wire Notes Line
 	5375 6000 575  6000
@@
 250 V AC MAX.
 NoConn ~ 4325 7075
+Wire Wire Line
+	10475 700  10225 700
+Wire Wire Line
+	10300 800  10300 1925
+Wire Wire Line
+	10300 800  10475 800
+Wire Wire Line
+	10300 1925 10475 1925
+Text Label 10325 1925 0    40   ~ 0
+NEUT
+Wire Wire Line
+	10300 1925 10300 3275
+Wire Wire Line
+	10300 3275 10475 3275
+Connection ~ 10300 1925
+Text Label 10325 3275 0    40   ~ 0
+NEUT
+Text Label 10325 4625 0    40   ~ 0
+NEUT
+Wire Wire Line
+	10300 3275 10300 4625
+Wire Wire Line
+	10300 4625 10475 4625
+Connection ~ 10300 3275
+Wire Wire Line
+	9900 2025 10475 2025
+Wire Wire Line
+	9900 3375 10475 3375
+Wire Wire Line
+	9900 4725 10475 4725
+Wire Wire Line
+	9900 1150 10225 1150
+Connection ~ 9900 1150
+Connection ~ 10225 1150
+Wire Wire Line
+	10225 700  10225 1150
+Wire Wire Line
+	9900 2500 10225 2500
+Connection ~ 9900 2500
+Connection ~ 10225 2500
+Wire Wire Line
+	10225 1150 10225 2500
+Wire Wire Line
+	10225 3850 9900 3850
+Connection ~ 9900 3850
+Wire Wire Line
+	10225 2500 10225 3850
+Text Notes 1400 4450 0    40   ~ 8
+INPUT POWER\n\nInput Power sources are :\na. Micro USB 5V to Wemos Lolin\nb. 28 V AC converted to 5 V via switching regulator\nc. 115 V AC converted to 5 V via wall wart or switching regulator\n\nWhen using option "b" or "c", the micro USB cable\nMUST be removed to prevent power conflicts.
+Text Label 2750 6675 0    40   ~ 0
+VCC
+Text Label 2975 6875 0    40   ~ 0
+SS
+Text Label 4350 6275 0    40   ~ 0
+LX
+Text Label 4325 7075 0    40   ~ 0
+R
+Text Label 2750 6275 0    40   ~ 0
+40VDC
+Wire Wire Line
+	2525 7625 2750 7625
+Wire Wire Line
+	5100 7500 5100 7400
+Wire Wire Line
+	5100 7400 4975 7400
+Connection ~ 4975 7400
+Wire Wire Line
+	4975 7400 4975 7625
+$Comp
+L wyostat:Jumper_NC_Small JP4
+U 1 1 5AE9DEF9
+P 2750 7475
+F 0 "JP4" V 2705 7552 50  0000 L CNN
+F 1 "GND" V 2795 7552 50  0000 L CNN
+F 2 "wyostat_fp:LED_0402" H 2750 7475 50  0001 C CNN
+F 3 "" H 2750 7475 50  0001 C CNN
+	1    2750 7475
+	0    1    1    0
+$EndComp
+Wire Wire Line
+	2750 7375 2750 7325
+Connection ~ 2750 7325
+Wire Wire Line
+	2750 7575 2750 7625
+Connection ~ 2750 7625
+Wire Wire Line
+	2750 7625 4475 7625
+Text Label 3100 7625 0    40   ~ 0
+GNDREF
+$Comp
+L wyostat:SCREW SC1
+U 1 1 5AED1CEA
+P 11000 5300
+F 0 "SC1" H 11085 5300 40  0000 L CNN
+F 1 "SCREW" H 11000 5400 40  0001 C CNN
+F 2 "wyostat_fp:MountingHole_3.2mm_M3_Pad_Via" H 11000 5300 60  0001 C CNN
+F 3 "" H 11000 5300 60  0000 C CNN
+	1    11000 5300
+	1    0    0    -1
+$EndComp
+$Comp
+L wyostat:SCREW SC2
+U 1 1 5AED2014
+P 11000 5600
+F 0 "SC2" H 11085 5600 40  0000 L CNN
+F 1 "SCREW" H 11000 5700 40  0001 C CNN
+F 2 "wyostat_fp:MountingHole_3.2mm_M3_Pad_Via" H 11000 5600 60  0001 C CNN
+F 3 "" H 11000 5600 60  0000 C CNN
+	1    11000 5600
+	1    0    0    -1
+$EndComp
+$Comp
+L wyostat:SCREW SC3
+U 1 1 5AED2111
+P 11000 5900
+F 0 "SC3" H 11085 5900 40  0000 L CNN
+F 1 "SCREW" H 11000 6000 40  0001 C CNN
+F 2 "wyostat_fp:MountingHole_3.2mm_M3_Pad_Via" H 11000 5900 60  0001 C CNN
+F 3 "" H 11000 5900 60  0000 C CNN
+	1    11000 5900
+	1    0    0    -1
+$EndComp
+$Comp
+L wyostat:SCREW SC4
+U 1 1 5AED2331
+P 11000 6200
+F 0 "SC4" H 11085 6200 40  0000 L CNN
+F 1 "SCREW" H 11000 6300 40  0001 C CNN
+F 2 "wyostat_fp:MountingHole_3.2mm_M3_Pad_Via" H 11000 6200 60  0001 C CNN
+F 3 "" H 11000 6200 60  0000 C CNN
+	1    11000 6200
+	1    0    0    -1
+$EndComp
 $EndSCHEMATC

Commit message: kicad PCB, track layout
Connections:
- wire segments 288 -> 291
Changed lines of the file:
@@
 Text Label 2225 825  0    40   ~ 0
 SW_M
-Text Label 750  825  2    40   ~ 0
+Text Label 750  1025 2    40   ~ 0
 IN1
 Text Label 750  925  2    40   ~ 0
 IN2
-Text Label 750  1025 2    40   ~ 0
+Text Label 750  825  2    40   ~ 0
 IN3
 Wire Wire Line
@@
 	1    0    0    -1
 $EndComp
+Wire Wire Line
+	2675 7550 2675 7400
+Wire Wire Line
+	2675 7400 2750 7325
+Wire Wire Line
+	2675 7550 2750 7625
 $EndSCHEMATC

Commit message: PCB layout, WIP
Parts:
- removed F2: Polyfuse, wyostat_fp:Fuse_SMD2920, symbol wyostat:Polyfuse
- removed J13, J15: AC_IN, wyostat_fp:TerminalBlock_Pheonix_MPT-2.54mm_2pol, symbol wyostat:Conn_01x02
- removed U6: Converter_AC_DC, wyostat_fp:Converter_AC_DC, symbol wyostat:Converter_AC_DC
- added C15: 4.7uF, wyostat_fp:C_0805, symbol wyostat:C_NP
- added D5: RClamp0854P.TCT, symbol wyostat:Diode_TVS
- added J13: USB_microAB, wyostat_fp:USB_Micro-B_Molex-105017-0001, symbol wyostat:USB_microAB
- added L2, L4: 330E, wyostat_fp:R_0805, symbol wyostat:IND_FERRITE_BEAD
- added L3: 90E, wyostat_fp:C_0805, symbol wyostat:IND_CHOKE_CM
- added R23: 0E, wyostat_fp:R_0805, symbol wyostat:R
- C2, C4, C6: DNP (none) -> DNP; manf# (none) -> Value
- J1: value PWR_In -> 24 V AC IN
- R12, R17, R5: DNP DNP -> -; manf# (none) -> Value
- R14, R2, R8: value 470 -> 0E; DNP (none) -> -
Connections:
- net labels added: 24Vac-C, 24Vac-H, D+, D-, ID, USB+, USB_D+, USB_D-, USB_ID
- net labels removed: LINE, NEUT
- wire segments 291 -> 322
- no-connect marks 12 -> 17
Other:
- note added: "1.5V"
- note added: "2V"
- note added: "5mA"
- note added: "INPUT POWER\n\nInput Power sources are :\na. Micro USB 5V to Wemos Lolin\nb. 28 V AC to 5 V DC via switching regulator\nc. 5 V via wall wart\n\nWhen using option "b" or "c", the micro USB cable\nMUST be removed to prevent power conflicts."
- note added: "USB INPUT + REGULATOR"
- note removed: "1.5V/5mA"
- note removed: "250 V AC MAX."
- note removed: "2V/5mA"
- note removed: "INPUT POWER\n\nInput Power sources are :\na. Micro USB 5V to Wemos Lolin\nb. 28 V AC converted to 5 V via switching regulator\nc. 115 V AC converted to 5 V via wall wart or switching regulator\n\nWhen using option "b" or "c", the micro USB cable\nMUST be removed to prevent power conflicts."
- moved on the sheet: C7, J1, J2, J3, J4, J5

Commit message: initial board layout
Parts:
- removed C8: 100nF, wyostat_fp:C_0805, symbol wyostat:C_NP
- removed D5: RClamp0854P.TCT, symbol wyostat:Diode_TVS
- removed J10: MOSI, wyostat_fp:Pin_Header_Straight_1x01, symbol wyostat:Conn_01x01
- removed J11: RST, wyostat_fp:Pin_Header_Straight_1x01, symbol wyostat:Conn_01x01
- removed J12: GND, wyostat_fp:Pin_Header_Straight_1x01, symbol wyostat:Conn_01x01
- removed J6: MISO, wyostat_fp:Pin_Header_Straight_1x01, symbol wyostat:Conn_01x01
- removed J7: 3V3, wyostat_fp:Pin_Header_Straight_1x01, symbol wyostat:Conn_01x01
- removed J8: SCK, wyostat_fp:Pin_Header_Straight_1x01, symbol wyostat:Conn_01x01
- removed J9: SPI, wyostat_fp:Pin_Header_Straight_2x03, symbol wyostat:Conn_02x03_Odd_Even
- removed L3: 90E, wyostat_fp:C_0805, symbol wyostat:IND_CHOKE_CM
- added D5: CDSOD323-T05L, Diodes_SMD:D_SOD-323_HandSoldering, symbol wyostat:1N5819
- added R24, R25: 0E, wyostat_fp:R_0805, symbol wyostat:R
- C10: footprint Capacitors_SMD:CP_Elec_10x10 -> wyostat_fp:CP_Elec_10x10
- Q1, Q2, Q3: footprint SMD_Packages:DPAK-2 -> wyostat_fp:DPAK-2
- R23: DNP (none) -> DNP
Connections:
- net D+: now also R24.2
- net D-: now also R23.2
- net GND: now also D5.2 (A)
- net ID: now also R25.2; no longer R23.2
- net USB+: now also D5.1 (K)
- net USB_D+: now also R24.1
- net USB_D-: now also R23.1
- net USB_ID: now also R25.1; no longer R23.1
- no-connect marks 17 -> 15
Other:
- note added: "INPUT POWER\n\nInput Power sources are :\na. Micro USB 5V to Wemos Lolin\nb. 28 V AC to 5 V DC via switching regulator\nc. Micro USB on Wyostat (only Power, no Data)\n\nWhen using option "b" or "c", the micro USB cable\nMUST be removed to prevent power conflicts.\n\nWhen using option "a", the Power Selector Header\nmust be in OFF position."
- note removed: "DECIDE how to couple 5V_IN to 5V"
- note removed: "INPUT POWER\n\nInput Power sources are :\na. Micro USB 5V to Wemos Lolin\nb. 28 V AC to 5 V DC via switching regulator\nc. 5 V via wall wart\n\nWhen using option "b" or "c", the micro USB cable\nMUST be removed to prevent power conflicts."
- note removed: "Native SPI pins are (clk, mosi, miso, cs):\nSPI1: 6, 8, 7, 11\nHSPI: 14,13,12,15\nVSPI: 18,23,19, 5\nIf using native pins max SPI clock can be set to 80 MHZ.\nOnly HSPI & VSPI are supported by esp-idf driver."
- note removed: "SPI HEADER"
- note removed: "SPI header with breakout pins.\nConnect with wire to appropriate\npins on ESP32"
- moved on the sheet: J16, SC1, SC2, SC3, SC4
